File: PickupPanel.brd (EAGLE design)
At the start: 128.5 x 30 mm, 3 parts

Commit message: Building the circuit
Changed lines of the file:
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@@
 <setting verticaltext="up"/>
 </settings>
-<grid distance="25" unitdist="mil" unit="mm" style="dots" multiple="1" display="no" altdistance="5" altunitdist="mil" altunit="mil"/>
+<grid distance="25" unitdist="mil" unit="mil" style="dots" multiple="1" display="no" altdistance="5" altunitdist="mil" altunit="mil"/>
 <layers>
 <layer number="1" name="Top" color="4" fill="1" visible="yes" active="yes"/>
@@
 <layer number="49" name="Reference" color="7" fill="1" visible="yes" active="yes"/>
 <layer number="50" name="dxf" color="7" fill="1" visible="no" active="no"/>
-<layer number="51" name="tDocu" color="7" fill="1" visible="yes" active="yes"/>
+<layer number="51" name="tDocu" color="12" fill="1" visible="yes" active="yes"/>
 <layer number="52" name="bDocu" color="7" fill="1" visible="yes" active="yes"/>
 <layer number="53" name="tGND_GNDA" color="7" fill="9" visible="no" active="no"/>
@@
 <rectangle x1="-0.635" y1="-0.635" x2="8.255" y2="30" layer="30"/>
 <rectangle x1="120.015" y1="-0.635" x2="128.905" y2="30" layer="30"/>
-<circle x="16.51" y="40.005" radius="6" width="0.4064" layer="51"/>
 <text x="21.59" y="27.94" size="1.778" layer="21" rot="SR270">In</text>
-<text x="35.56" y="27.94" size="1.778" layer="21" rot="SR270">Gain</text>
-<text x="21.59" y="12.7" size="1.778" layer="21" rot="SR270">Clean</text>
-<text x="34.925" y="12.065" size="1.778" layer="21" rot="SR270">Fuzz</text>
+<text x="35.56" y="10.16" size="1.778" layer="21" rot="SR270">Gain</text>
+<text x="20.32" y="12.065" size="1.778" layer="21" rot="SR270">Clean</text>
+<text x="35.56" y="26.67" size="1.778" layer="21" rot="SR270">Fuzz</text>
 </plain>
 <attributes>
@@
 </elements>
 <signals>
+<signal name="N$2">
+<via x="15.195" y="8.755" extent="1-16" drill="6"/>
+<via x="29.8" y="8.015" extent="1-16" drill="7.1"/>
+<via x="15.83" y="22.725" extent="1-16" drill="9.6012"/>
+<wire x1="15.195" y1="8.755" x2="29.8" y2="8.015" width="0" layer="19" extent="1-1"/>
+<wire x1="15.83" y1="22.725" x2="15.195" y2="8.755" width="0" layer="19" extent="1-1"/>
+</signal>
 <signal name="GND">
-<via x="15.83" y="22.725" extent="1-16" drill="9.6012"/>
-<via x="29.165" y="22.725" extent="1-16" drill="7.1"/>
 <polygon width="0.8128" layer="16">
-<vertex x="0" y="31.75"/>
-<vertex x="131.445" y="32.385"/>
+<vertex x="-8.89" y="36.195"/>
+<vertex x="132.715" y="35.56"/>
 <vertex x="131.445" y="-0.635"/>
 <vertex x="-1.27" y="-1.27"/>
 </polygon>
-<wire x1="15.83" y1="22.725" x2="29.165" y2="22.725" width="0" layer="19" extent="1-1"/>
-<via x="29.8" y="9.39" extent="1-16" drill="7.1"/>
-<via x="15.195" y="9.39" extent="1-16" drill="6"/>
+</signal>
+<signal name="GND1">
+<via x="29.8" y="23.36" extent="1-16" drill="6"/>
 </signal>
 </signals>

Commit message: Completed first layout
Parts:
- moved U$1 1.27 mm to (78.1, 16.3)
Routing:
- net N$34: track 0.00 -> 88.9 mm
- net N$6: track 0.00 -> 56.1 mm
- net N$5: track 0.00 -> 54.8 mm
- net N$22: track 0.00 -> 46.8 mm
- net N$4: track 0.00 -> 45.0 mm
- net N$16: track 0.00 -> 44.9 mm
- net N$24: track 0.00 -> 41.7 mm
- net N$19: track 0.00 -> 38.4 mm
- net N$1: track 0.00 -> 37.9 mm
- net N$31: track 0.00 -> 33.8 mm
- net N$20: track 0.00 -> 33.2 mm
- net N$3: track 0.00 -> 32.8 mm
- net N$35: track 0.00 -> 31.8 mm
- net N$17: track 0.00 -> 28.4 mm
- net N$9: track 0.00 -> 25.0 mm
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Other:
- board text removed: "Clean"
- board text removed: "Fuzz"
- board text removed: "Gain"
- board text removed: "In"
