File: Hardware/PickupBoard.sch (EAGLE design)
At the start: 31 parts, among them U2 TL074_

Commit message: roughly on the board not routed
Parts:
- C3, C6, C7: device we-rcl:CAPACITOR-0603 -> TomW:C-EU050-024X044
Connections:
- net GAIN_IN: now also R1.1, R2.1; no longer R1.2, R2.2
- net GND: now also R1.2; no longer R1.1
- net N$15: now also R12.2; no longer R12.1
- net N$17: now also R12.1; no longer R12.2
- net N$2: now also R2.2; no longer R2.1
Other:
- moved on the sheet: R1, R12, R2
Changed lines of the file:
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@@
 <part name="R5" library="MusicThingModular" deviceset="RESISTOR" device="7MM" value="10k"/>
 <part name="R6" library="MusicThingModular" deviceset="RESISTOR" device="7MM" value="10K"/>
-<part name="C3" library="we-rcl" deviceset="CAPACITOR" device="-0603" value="47n"/>
-<part name="C6" library="we-rcl" deviceset="CAPACITOR" device="-0603" value="330pf"/>
+<part name="C3" library="TomW" deviceset="C-EU" device="050-024X044" value="47n"/>
+<part name="C6" library="TomW" deviceset="C-EU" device="050-024X044" value="330pf"/>
 <part name="SUPPLY1" library="supply2" deviceset="GND" device=""/>
 <part name="SUPPLY4" library="supply2" deviceset="GND" device=""/>
 <part name="SUPPLY5" library="supply2" deviceset="GND" device=""/>
 <part name="R7" library="MusicThingModular" deviceset="RESISTOR" device="7MM" value="10K"/>
-<part name="C7" library="we-rcl" deviceset="CAPACITOR" device="-0603" value="330pf"/>
+<part name="C7" library="TomW" deviceset="C-EU" device="050-024X044" value="330pf"/>
 <part name="R8" library="MusicThingModular" deviceset="RESISTOR" device="7MM" value="150k"/>
 <part name="R9" library="MusicThingModular" deviceset="RESISTOR" device="7MM" value="32k"/>
@@
 <instance part="JP3" gate="G$1" x="38.1" y="119.38"/>
 <instance part="JP4" gate="G$1" x="38.1" y="106.68"/>
-<instance part="R1" gate="G$1" x="111.76" y="177.8" rot="R90"/>
-<instance part="R2" gate="G$1" x="132.08" y="190.5" rot="R180"/>
+<instance part="R1" gate="G$1" x="111.76" y="177.8" rot="R270"/>
+<instance part="R2" gate="G$1" x="132.08" y="190.5"/>
 <instance part="R4" gate="G$1" x="154.94" y="160.02" rot="R90"/>
 <instance part="R5" gate="G$1" x="193.04" y="162.56" rot="R270"/>
 <instance part="R6" gate="G$1" x="147.32" y="101.6" rot="R180"/>
-<instance part="C3" gate="C" x="160.02" y="172.72"/>
-<instance part="C6" gate="C" x="180.34" y="172.72"/>
+<instance part="C3" gate="G$1" x="160.02" y="172.72" rot="R90"/>
+<instance part="C6" gate="G$1" x="180.34" y="172.72" rot="R90"/>
 <instance part="U2" gate="A" x="177.8" y="187.96"/>
 <instance part="U2" gate="C" x="251.46" y="99.06"/>
@@
 <instance part="SUPPLY5" gate="GND" x="167.64" y="60.96"/>
 <instance part="R7" gate="G$1" x="187.96" y="101.6" rot="R180"/>
-<instance part="C7" gate="C" x="251.46" y="86.36"/>
+<instance part="C7" gate="G$1" x="251.46" y="86.36" rot="R90"/>
 <instance part="R8" gate="G$1" x="251.46" y="73.66" rot="R180"/>
 <instance part="R9" gate="G$1" x="226.06" y="73.66" rot="R90"/>
@@
 <instance part="U2" gate="D" x="320.04" y="180.34"/>
 <instance part="R10" gate="G$1" x="215.9" y="187.96" rot="R180"/>
-<instance part="R12" gate="G$1" x="200.66" y="147.32" rot="R270"/>
+<instance part="R12" gate="G$1" x="200.66" y="147.32" rot="R90"/>
 <instance part="R13" gate="G$1" x="330.2" y="99.06" rot="R180"/>
 <instance part="D2" gate="G$1" x="157.48" y="78.74" rot="R90"/>
@@
 </segment>
 <segment>
-<pinref part="R1" gate="G$1" pin="1"/>
+<pinref part="R1" gate="G$1" pin="2"/>
 <wire x1="111.76" y1="165.1" x2="111.76" y2="172.72" width="0.1524" layer="91"/>
 <pinref part="SUPPLY1" gate="GND" pin="GND"/>
@@
 <net name="GAIN_IN" class="0">
 <segment>
-<pinref part="R1" gate="G$1" pin="2"/>
+<pinref part="R1" gate="G$1" pin="1"/>
 <wire x1="111.76" y1="182.88" x2="111.76" y2="190.5" width="0.1524" layer="91"/>
 <junction x="111.76" y="190.5"/>
-<pinref part="R2" gate="G$1" pin="2"/>
+<pinref part="R2" gate="G$1" pin="1"/>
 <wire x1="127" y1="190.5" x2="111.76" y2="190.5" width="0.1524" layer="91"/>
 <pinref part="U$1" gate="G$1" pin="3"/>
@@
 <net name="N$2" class="0">
 <segment>
-<pinref part="R2" gate="G$1" pin="1"/>
+<pinref part="R2" gate="G$1" pin="2"/>
 <pinref part="U2" gate="A" pin="+IN"/>
 <wire x1="170.18" y1="190.5" x2="137.16" y2="190.5" width="0.1524" layer="91"/>
@@
 <segment>
 <wire x1="167.64" y1="185.42" x2="167.64" y2="172.72" width="0.1524" layer="91"/>
-<pinref part="C6" gate="C" pin="1"/>
+<pinref part="C6" gate="G$1" pin="1"/>
 <wire x1="177.8" y1="172.72" x2="167.64" y2="172.72" width="0.1524" layer="91"/>
 <junction x="167.64" y="172.72"/>
 <wire x1="167.64" y1="172.72" x2="167.64" y2="147.32" width="0.1524" layer="91"/>
-<pinref part="C3" gate="C" pin="2"/>
-<wire x1="162.56" y1="172.72" x2="167.64" y2="172.72" width="0.1524" layer="91"/>
+<pinref part="C3" gate="G$1" pin="2"/>
+<wire x1="165.1" y1="172.72" x2="167.64" y2="172.72" width="0.1524" layer="91"/>
 <pinref part="U2" gate="A" pin="-IN"/>
 <wire x1="170.18" y1="185.42" x2="167.64" y2="185.42" width="0.1524" layer="91"/>
@@
 <net name="N$7" class="0">
 <segment>
-<pinref part="C3" gate="C" pin="1"/>
+<pinref part="C3" gate="G$1" pin="1"/>
 <pinref part="R4" gate="G$1" pin="2"/>
 <wire x1="157.48" y1="172.72" x2="154.94" y2="172.72" width="0.1524" layer="91"/>
@@
 <wire x1="243.84" y1="96.52" x2="238.76" y2="96.52" width="0.1524" layer="91"/>
 <wire x1="238.76" y1="96.52" x2="238.76" y2="86.36" width="0.1524" layer="91"/>
-<pinref part="C7" gate="C" pin="1"/>
+<pinref part="C7" gate="G$1" pin="1"/>
 <wire x1="238.76" y1="86.36" x2="238.76" y2="73.66" width="0.1524" layer="91"/>
 <wire x1="248.92" y1="86.36" x2="238.76" y2="86.36" width="0.1524" layer="91"/>
@@
 <wire x1="259.08" y1="99.06" x2="264.16" y2="99.06" width="0.1524" layer="91"/>
 <wire x1="264.16" y1="99.06" x2="264.16" y2="86.36" width="0.1524" layer="91"/>
-<pinref part="C7" gate="C" pin="2"/>
+<pinref part="C7" gate="G$1" pin="2"/>
 <wire x1="264.16" y1="86.36" x2="264.16" y2="73.66" width="0.1524" layer="91"/>
-<wire x1="254" y1="86.36" x2="264.16" y2="86.36" width="0.1524" layer="91"/>
+<wire x1="256.54" y1="86.36" x2="264.16" y2="86.36" width="0.1524" layer="91"/>
 <junction x="264.16" y="86.36"/>
 <pinref part="R8" gate="G$1" pin="1"/>
@@
 <wire x1="185.42" y1="187.96" x2="193.04" y2="187.96" width="0.1524" layer="91"/>
 <wire x1="193.04" y1="187.96" x2="193.04" y2="172.72" width="0.1524" layer="91"/>
-<pinref part="C6" gate="C" pin="2"/>
+<pinref part="C6" gate="G$1" pin="2"/>
 <wire x1="193.04" y1="172.72" x2="193.04" y2="167.64" width="0.1524" layer="91"/>
-<wire x1="182.88" y1="172.72" x2="193.04" y2="172.72" width="0.1524" layer="91"/>
+<wire x1="185.42" y1="172.72" x2="193.04" y2="172.72" width="0.1524" layer="91"/>
 <junction x="193.04" y="172.72"/>
 <pinref part="R5" gate="G$1" pin="1"/>
 <junction x="193.04" y="187.96"/>
 <wire x1="193.04" y1="172.72" x2="200.66" y2="172.72" width="0.1524" layer="91"/>
-<pinref part="R12" gate="G$1" pin="1"/>
+<pinref part="R12" gate="G$1" pin="2"/>
 <wire x1="200.66" y1="152.4" x2="200.66" y2="172.72" width="0.1524" layer="91"/>
 <wire x1="210.82" y1="187.96" x2="193.04" y2="187.96" width="0.1524" layer="91"/>
@@
 <wire x1="99.06" y1="119.38" x2="99.06" y2="104.14" width="0.1524" layer="91"/>
 <wire x1="99.06" y1="104.14" x2="104.14" y2="104.14" width="0.1524" layer="91"/>
-<pinref part="R12" gate="G$1" pin="2"/>
+<pinref part="R12" gate="G$1" pin="1"/>
 <wire x1="200.66" y1="142.24" x2="200.66" y2="119.38" width="0.1524" layer="91"/>
 </segment>

Commit message: Designed and routed
Parts:
- removed C3: 47n, TomW:C-EU050-024X044
- removed JP2: POT, SparkFun-Connectors:M02LOCK
- removed R4: 10k, MusicThingModular:RESISTOR7MM
- added CLN, GRND: M01PTH, SparkFun-Connectors:M01PTH
- C6, C7: device TomW:C-EU050-024X044 -> gm-caps-ceramic:050X030_0251
- JP1: value INOUT -> (none); device SparkFun-Connectors:M03LOCK -> SparkFun-Connectors:M03PTH
Connections:
- removed net N$13: R13.2
- removed net N$16: JP1.2, R10.1
- removed net N$19: JP1.1, R13.1
- removed net N$4: C3.2, C6.1, JP2.2, U2A.-IN
- removed net N$6: JP2.1, R5.2
- removed net N$7: C3.1, R4.2
- new net CLEAN: CLN.1, R10.2
- new net END: C6.1, JP1.2, U2C.-IN
- new net FUZZ: JP1.3, R13.2
- new net WIPER: JP1.1, R5.1
- net -12V: now also C5.1; no longer C5.2
- net GAIN_IN: now also R1.2, R2.2; no longer R1.1, R2.1
- net GND: now also C5.2, GRND.1, R1.1; no longer C5.1, JP1.3, R1.2, R4.1
- net N$11: now also R8.1, U2A.-IN; no longer R8.2, U2C.-IN
- net N$12: now also R13.1, R8.2, U2A.OUT; no longer R8.1, U2C.OUT
- net N$15: now also R10.1, R5.2, U2C.OUT; no longer R10.2, R5.1, U2A.OUT
- net N$2: now also R2.1, U2C.+IN; no longer R2.2, U2A.+IN
- net N$8: now also R7.2, U2A.+IN; no longer R7.1, U2C.+IN
- net N$9: now also R7.1; no longer R7.2
Other:
- moved on the sheet: C5, C6, C7, JP1, R1, R10, R13, R2, R5, R7, R8, U2A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
