File: Hardware/PickupDaughterBoard.brd (EAGLE design)
At the start: 28.3 x 29 mm, 5 parts

Commit message: First rev5 upload
Parts:
- GAIN: value 50k -> B1M
Changed lines of the file:
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@@
 <attribute name="NAME" x="5.207" y="1.905" size="1.016" layer="25" rot="SR180"/>
 </element>
-<element name="GAIN" library="TomW" package="EVUF" value="50k" x="22.86" y="5.715" smashed="yes" rot="R270">
+<element name="GAIN" library="TomW" package="EVUF" value="B1M" x="22.86" y="5.715" smashed="yes" rot="R270">
 <attribute name="NAME" x="26.574" y="8.969" size="1.27" layer="25" rot="R270"/>
 <attribute name="VALUE" x="17.678" y="5.516" size="1.27" layer="27" rot="R270"/>

Commit message: Designed and routed
Parts:
- removed JP3: (no value), SparkFun-Connectors:1X03_LOCK
- added C3: 47n, TomW:C050-024X044
- added CLN, GRND: M01PTH, SparkFun-Connectors:1X01
- added R4: 10k, MusicThingModular:VERTICAL_RESISTOR
- added U$1: SUBMINI_SPDT, MusicThingModular:SUBMINI_TOGGLE
- added U$2: (no value), MusicThingModular:SINGLE_COIL_CUTOUT_MILLING
- JP2: value M02LOCK -> (none); device SparkFun-Connectors:1X02_LOCK -> SparkFun-Connectors:1X03
- moved JP2 6.73 mm to (26.7, 11.7)
- turned FUZZ to 90 degrees
Connections:
- net N$8 renamed WIPER
- removed net N$1: FUZZ.P$1_TIP, JP3.1
- removed net N$2: CLEAN.P$1_TIP, JP3.2
- removed net N$4: GAIN.1, JP2.2
- new net CLEAN: CLEAN.P$1_TIP, CLN.1
- new net END: C3.1, GAIN.1, JP2.2, U$1.3
- new net FUZZ: FUZZ.P$1_TIP, JP2.3
- new net N$7: C3.2, R4.2, U$1.COM
- net GND: now also GRND.1, R4.1; no longer JP3.3
Routing:
- net N$2: track 51.1 -> 0.00 mm
- net END: track 0.00 -> 49.0 mm
- net N$7: track 0.00 -> 22.8 mm
- net N$1: track 21.5 -> 0.00 mm
- net N$4: track 14.1 -> 0.00 mm
- net CLEAN: track 0.00 -> 13.0 mm
- net FUZZ: track 0.00 -> 11.8 mm
- net WIPER: track 14.3 -> 17.5 mm
Other:
- board size 28.3 x 29 mm -> 71 x 18.4 mm
- board text added: "Music Thing Modular Pickup Daughterboard August 2017 PCB Rev 2 BY-CC-SA"
- board text removed: "Music Thing Modular Pickup Daughterboard September 2015 PCB Rev 1 BY-CC-SA"

Commit message: Rev5  with gerbers
Parts:
- removed U$2: (no value), MusicThingModular:SINGLE_COIL_CUTOUT_MILLING
Routing:
- net CLEAN: track 13.0 -> 13.9 mm
Other:
- board size 71 x 18.4 mm -> 35.2 x 27.3 mm
- board text added: "Music Thing Modular Electrophone Daughterboard August 2017 PCB Rev 5 BY-CC-SA"
- board text removed: "Music Thing Modular Pickup Daughterboard August 2017 PCB Rev 2 BY-CC-SA"
